File: RGBBoard/rgbboard.sch (EAGLE design)
At the start: 33 parts, among them J1 BOOT, J2 5.5x2.1mm Barrel, U1 MIC5219 5V, U2 ATMEGA328P_TQFP, U3 V_REG_317SMD, Y1 16MHz

Commit message: Layout Done - Need to Pass DRC
Parts:
- J3: value (none) -> ESP
- J4: value (none) -> PROG
Other:
- note removed: "ESP Connector Headers"
Changed lines of the file:
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@@
 <part name="GND13" library="SparkFun-PowerSymbols" deviceset="GND" device=""/>
 <part name="SUPPLY7" library="SparkFun-PowerSymbols" deviceset="3.3V" device=""/>
-<part name="J3" library="SparkFun-Connectors" deviceset="CONN_04X2" device=""/>
+<part name="J3" library="SparkFun-Connectors" deviceset="CONN_04X2" device="" value="ESP"/>
 <part name="GND14" library="SparkFun-PowerSymbols" deviceset="GND" device=""/>
 <part name="SUPPLY6" library="SparkFun-PowerSymbols" deviceset="3.3V" device=""/>
@@
 <part name="GND18" library="SparkFun-PowerSymbols" deviceset="GND" device=""/>
 <part name="GND19" library="SparkFun-PowerSymbols" deviceset="GND" device=""/>
-<part name="J4" library="SparkFun-Connectors" deviceset="6_PIN_SERIAL_TARGET" device=""/>
+<part name="J4" library="SparkFun-Connectors" deviceset="6_PIN_SERIAL_TARGET" device="" value="PROG"/>
 <part name="J1" library="SparkFun-Connectors" deviceset="CONN_04" device="" value="BOOT"/>
 </parts>
@@
 <sheet>
 <plain>
-<text x="200.66" y="50.8" size="1.778" layer="91">ESP Connector Headers</text>
 </plain>
 <instances>
@@
 </segment>
 <segment>
+<pinref part="J4" gate="G$1" pin="GND"/>
 <pinref part="J4" gate="G$1" pin="CTS"/>
-<pinref part="J4" gate="G$1" pin="GND"/>
-<wire x1="177.8" y1="63.5" x2="177.8" y2="66.04" width="0.1524" layer="91"/>
+<wire x1="177.8" y1="66.04" x2="177.8" y2="63.5" width="0.1524" layer="91"/>
+<pinref part="GND11" gate="1" pin="GND"/>
 <wire x1="177.8" y1="66.04" x2="177.8" y2="71.12" width="0.1524" layer="91"/>
-<pinref part="GND11" gate="1" pin="GND"/>
+<junction x="177.8" y="66.04"/>
 </segment>
 </net>
@@
 <pinref part="C8" gate="G$1" pin="1"/>
 <wire x1="15.24" y1="106.68" x2="20.32" y2="106.68" width="0.1524" layer="91"/>
+<wire x1="20.32" y1="106.68" x2="20.32" y2="86.36" width="0.1524" layer="91"/>
+<pinref part="D6" gate="G$1" pin="VDD"/>
+<wire x1="20.32" y1="86.36" x2="20.32" y2="66.04" width="0.1524" layer="91"/>
+<wire x1="20.32" y1="66.04" x2="20.32" y2="45.72" width="0.1524" layer="91"/>
+<wire x1="20.32" y1="45.72" x2="20.32" y2="25.4" width="0.1524" layer="91"/>
+<wire x1="20.32" y1="25.4" x2="27.94" y2="25.4" width="0.1524" layer="91"/>
+<pinref part="C12" gate="G$1" pin="1"/>
+<wire x1="15.24" y1="25.4" x2="20.32" y2="25.4" width="0.1524" layer="91"/>
+<junction x="20.32" y="25.4"/>
+<pinref part="C11" gate="G$1" pin="1"/>
+<wire x1="15.24" y1="45.72" x2="20.32" y2="45.72" width="0.1524" layer="91"/>
+<junction x="20.32" y="45.72"/>
+<pinref part="D5" gate="G$1" pin="VDD"/>
+<wire x1="20.32" y1="45.72" x2="27.94" y2="45.72" width="0.1524" layer="91"/>
+<pinref part="C10" gate="G$1" pin="1"/>
+<wire x1="15.24" y1="66.04" x2="20.32" y2="66.04" width="0.1524" layer="91"/>
+<junction x="20.32" y="66.04"/>
+<pinref part="D4" gate="G$1" pin="VDD"/>
+<wire x1="20.32" y1="66.04" x2="27.94" y2="66.04" width="0.1524" layer="91"/>
+<pinref part="C9" gate="G$1" pin="1"/>
+<wire x1="15.24" y1="86.36" x2="20.32" y2="86.36" width="0.1524" layer="91"/>
+<junction x="20.32" y="86.36"/>
 <pinref part="D3" gate="G$1" pin="VDD"/>
-<wire x1="15.24" y1="86.36" x2="20.32" y2="86.36" width="0.1524" layer="91"/>
-<pinref part="C9" gate="G$1" pin="1"/>
-<wire x1="27.94" y1="86.36" x2="20.32" y2="86.36" width="0.1524" layer="91"/>
-<wire x1="20.32" y1="106.68" x2="20.32" y2="86.36" width="0.1524" layer="91"/>
-<pinref part="D4" gate="G$1" pin="VDD"/>
-<wire x1="15.24" y1="66.04" x2="20.32" y2="66.04" width="0.1524" layer="91"/>
-<pinref part="C10" gate="G$1" pin="1"/>
-<wire x1="20.32" y1="66.04" x2="27.94" y2="66.04" width="0.1524" layer="91"/>
-<wire x1="20.32" y1="86.36" x2="20.32" y2="66.04" width="0.1524" layer="91"/>
-<pinref part="D5" gate="G$1" pin="VDD"/>
-<wire x1="15.24" y1="45.72" x2="20.32" y2="45.72" width="0.1524" layer="91"/>
-<pinref part="C11" gate="G$1" pin="1"/>
-<wire x1="20.32" y1="45.72" x2="27.94" y2="45.72" width="0.1524" layer="91"/>
-<wire x1="20.32" y1="66.04" x2="20.32" y2="45.72" width="0.1524" layer="91"/>
-<pinref part="D6" gate="G$1" pin="VDD"/>
-<wire x1="15.24" y1="25.4" x2="20.32" y2="25.4" width="0.1524" layer="91"/>
-<pinref part="C12" gate="G$1" pin="1"/>
-<wire x1="20.32" y1="25.4" x2="27.94" y2="25.4" width="0.1524" layer="91"/>
-<wire x1="20.32" y1="45.72" x2="20.32" y2="25.4" width="0.1524" layer="91"/>
-</segment>
-<segment>
+<wire x1="20.32" y1="86.36" x2="27.94" y2="86.36" width="0.1524" layer="91"/>
+</segment>
+<segment>
